Commit message: remove velocity control

File: gym_panda/panda_bullet/assets/franka_panda/panda.urdf (robot description, URDF)
Before this commit: robot panda, 13 links, 12 joints
Joints:
- joint panda_joint1: axis (none) -> 0 0 1; limit (none) -> lower=-2.9671 upper=2.9671 effort=87 velocity=2.1750; type fixed -> revolute
- joint panda_joint3: axis (none) -> 0 0 1; limit (none) -> lower=-2.9671 upper=2.9671 effort=87 velocity=2.1750; type fixed -> revolute
- joint panda_joint5: axis (none) -> 0 0 1; limit (none) -> lower=-2.9671 upper=2.9671 effort=12 velocity=2.6100; type fixed -> revolute
- joint panda_joint7: axis (none) -> 0 0 1; limit (none) -> lower=-2.9671 upper=2.9671 effort=12 velocity=2.6100; type fixed -> revolute
